File: hardware/workbench-r03/workbench-r03.kicad_pcb (KiCad board)
At the start: 4 copper layers, 126 x 105 mm, 62 parts, among them J1 USB-C USB2.0, J2 DISPLAY HARNESS - SEE README, J3 SWD 3V3 GND SWDIO SWCLK, J4 AUX GND 3V3 GP0 GP23 GP29, SW1 KEY_1 MX HOTSWAP, SW10 KEY_10 MX HOTSWAP, SW11 KEY_11 MX HOTSWAP, SW12 KEY_12 MX HOTSWAP, SW13 KEY_13 MX HOTSWAP, SW14 KEY_14 MX HOTSWAP, SW15 KEY_15 MX HOTSWAP, SW16 KEY_16 MX HOTSWAP, SW17 KEY_17 MX HOTSWAP, SW18 KEY_18 MX HOTSWAP, SW19 BOOTSEL, SW2 KEY_2 MX HOTSWAP, SW20 RESET, SW3 KEY_3 MX HOTSWAP, SW4 KEY_4 MX HOTSWAP, SW5 KEY_5 MX HOTSWAP, SW6 KEY_6 MX HOTSWAP, SW7 KEY_7 MX HOTSWAP, SW8 KEY_8 MX HOTSWAP, SW9 KEY_9 MX HOTSWAP, U1 RP2040, U2 W25Q128JVSIQ / 16MiB, U3 AP2112K-3.3, U4 USBLC6-2SC6, Y1 12MHz ABM8-272-T3

Commit message: Improve keypad layout configuration and device profile handling
Parts:
- added J5: EXTERNAL BOOT BUTTON, PinHeader_1x02_P2.54mm_Vertical, F.Cu at (147.5, 54.0)
- added J6: EXTERNAL RESET BUTTON, PinHeader_1x02_P2.54mm_Vertical, F.Cu at (154.0, 54.0)
- J4: value AUX GND 3V3 GP0 GP23 GP29 -> EXPANSION / 3V3 IO; footprint PinHeader_1x05_P2.54mm_Vertical -> PinHeader_1x07_P2.54mm_Vertical
- moved J4 84.1 mm to (60.0, 53.0)
Connections:
- J4 pad 5: /GPIO29 -> /GPIO24
- U1 pad 36: (no net) -> /GPIO24
- U1 pad 37: (no net) -> /GPIO25
Other:
- board text added: "BOOT"
- board text added: "GP0"
- board text added: "GP23"
- board text added: "GP24"
- board text added: "GP25"
- board text added: "GP29"
- board text added: "J4 / 3V3 IO"
- board text added: "RESET"
