File: hardware/workbench-r03/workbench-r03.kicad_sch (KiCad schematic)
At the start: 57 parts, among them J1 USB-C USB2.0, J2 DISPLAY HARNESS - SEE README, J3 SWD 3V3 GND SWDIO SWCLK, J4 AUX GND 3V3 GP0 GP23 GP29, SW1 KEY_1 MX HOTSWAP, SW10 KEY_10 MX HOTSWAP, SW11 KEY_11 MX HOTSWAP, SW12 KEY_12 MX HOTSWAP, SW13 KEY_13 MX HOTSWAP, SW14 KEY_14 MX HOTSWAP, SW15 KEY_15 MX HOTSWAP, SW16 KEY_16 MX HOTSWAP, SW17 KEY_17 MX HOTSWAP, SW18 KEY_18 MX HOTSWAP, SW19 BOOTSEL, SW2 KEY_2 MX HOTSWAP, SW20 RESET, SW3 KEY_3 MX HOTSWAP, SW4 KEY_4 MX HOTSWAP, SW5 KEY_5 MX HOTSWAP, SW6 KEY_6 MX HOTSWAP, SW7 KEY_7 MX HOTSWAP, SW8 KEY_8 MX HOTSWAP, SW9 KEY_9 MX HOTSWAP, U1 RP2040, U2 W25Q128JVSIQ / 16MiB, U3 AP2112K-3.3, U4 USBLC6-2SC6, Y1 12MHz ABM8-272-T3

Commit message: Improve keypad layout configuration and device profile handling
Parts:
- added J5: EXTERNAL BOOT BUTTON, Connector_PinHeader_2.54mm:PinHeader_1x02_P2.54mm_Vertical, symbol Connector_Generic:Conn_01x02
- added J6: EXTERNAL RESET BUTTON, Connector_PinHeader_2.54mm:PinHeader_1x02_P2.54mm_Vertical, symbol Connector_Generic:Conn_01x02
- J4: value AUX GND 3V3 GP0 GP23 GP29 -> EXPANSION / 3V3 IO; footprint Connector_PinHeader_2.54mm:PinHeader_1x05_P2.54mm_Vertical -> Connector_PinHeader_2.54mm:PinHeader_1x07_P2.54mm_Vertical; symbol Connector_Generic:Conn_01x05 -> Connector_Generic:Conn_01x07
Connections:
- net BOOT_BUTTON: now also J5.1 (Pin_1)
- net GND: now also J5.2 (Pin_2), J6.2 (Pin_2)
- net GPIO29: now also J4.7 (Pin_7); no longer J4.5 (Pin_5)
- net RUN: now also J6.1 (Pin_1)
- net GPIO24: now reaches U1.36 (GPIO24)
- net GPIO24: now also J4.5 (Pin_5)
- net GPIO25: now reaches U1.37 (GPIO25)
- net GPIO25: now also J4.6 (Pin_6)
- no-connect marks 5 -> 3
