File: hardware/workbench-s3-r01/workbench-s3-r01.kicad_sch (KiCad schematic)
At the start: 52 parts, among them J1 YD P1 / RIGHT SOCKET / 1x22, J2 DISPLAY / MODULE PIN 1 = 3V3, J4 EXPANSION / 22 SPARE GPIO / 3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, J5 EXTERNAL BOOT / GPIO0 TO GND, J6 EXTERNAL RESET / EN TO GND, J7 YD P2 / LEFT SOCKET / 1x22, J8 LOWER / I2C4 TO J9 / 1:1, J9 UPPER / I2C4 TO J8 / 1:1, SW1 KEY_1 MX HOTSWAP, SW10 KEY_10 MX HOTSWAP, SW11 KEY_11 MX HOTSWAP, SW12 KEY_12 MX HOTSWAP, SW13 KEY_13 MX HOTSWAP, SW14 KEY_14 MX HOTSWAP, SW15 KEY_15 MX HOTSWAP, SW16 KEY_16 MX HOTSWAP, SW17 KEY_17 MX HOTSWAP, SW18 KEY_18 MX HOTSWAP, SW2 KEY_2 MX HOTSWAP, SW3 KEY_3 MX HOTSWAP, SW4 KEY_4 MX HOTSWAP, SW5 KEY_5 MX HOTSWAP, SW6 KEY_6 MX HOTSWAP, SW7 KEY_7 MX HOTSWAP, SW8 KEY_8 MX HOTSWAP, SW9 KEY_9 MX HOTSWAP, U1 MCP23017-E/SO / 0x20

Commit message: Update device profile layouts and supporting resources
Parts:
- removed C1: 10u 10V X7R, Capacitor_SMD:C_0805_2012Metric_Pad1.18x1.45mm_HandSolder, symbol Device:C
- removed C2: 100n 16V X7R, Capacitor_SMD:C_0805_2012Metric_Pad1.18x1.45mm_HandSolder, symbol Device:C
- removed C3: 100n 16V X7R / U1, Capacitor_SMD:C_0805_2012Metric_Pad1.18x1.45mm_HandSolder, symbol Device:C
- removed D1, D10, D11, D12, D13, D14, D15, D16, D17, D18, D2, D3, D4, D5, D6, D7, D8, D9: 1N4148W / K TO ROW, Diode_SMD:D_SOD-123, symbol Device:D
- removed J2: DISPLAY / MODULE PIN 1 = 3V3, Connector_PinHeader_2.54mm:PinHeader_1x09_P2.54mm_Vertical, symbol Connector_Generic:Conn_01x09
- removed J9: UPPER / I2C4 TO J8 / 1:1, Connector_JST:JST_XH_B4B-XH-A_1x04_P2.50mm_Vertical, symbol Connector_Generic:Conn_01x04
- removed R1, R2: 2.2k I2C PULLUP, Resistor_SMD:R_0805_2012Metric_Pad1.20x1.40mm_HandSolder, symbol Device:R
- removed R4: 10k U1 RESET PULLUP, Resistor_SMD:R_0805_2012Metric_Pad1.20x1.40mm_HandSolder, symbol Device:R
- removed SW1: KEY_1 MX HOTSWAP, Workbench:keyswitch_cherrymx_hotswap_1u, symbol Switch:SW_Push
- removed SW10: KEY_10 MX HOTSWAP, Workbench:keyswitch_cherrymx_hotswap_1u, symbol Switch:SW_Push
- removed SW11: KEY_11 MX HOTSWAP, Workbench:keyswitch_cherrymx_hotswap_1u, symbol Switch:SW_Push
- removed SW12: KEY_12 MX HOTSWAP, Workbench:keyswitch_cherrymx_hotswap_1u, symbol Switch:SW_Push
- removed SW13: KEY_13 MX HOTSWAP, Workbench:keyswitch_cherrymx_hotswap_1u, symbol Switch:SW_Push
- removed SW14: KEY_14 MX HOTSWAP, Workbench:keyswitch_cherrymx_hotswap_1u, symbol Switch:SW_Push
- removed SW15: KEY_15 MX HOTSWAP, Workbench:keyswitch_cherrymx_hotswap_1u, symbol Switch:SW_Push
- removed SW16: KEY_16 MX HOTSWAP, Workbench:keyswitch_cherrymx_hotswap_1u, symbol Switch:SW_Push
- removed SW17: KEY_17 MX HOTSWAP, Workbench:keyswitch_cherrymx_hotswap_1u, symbol Switch:SW_Push
- removed SW18: KEY_18 MX HOTSWAP, Workbench:keyswitch_cherrymx_hotswap_1u, symbol Switch:SW_Push
- removed SW2: KEY_2 MX HOTSWAP, Workbench:keyswitch_cherrymx_hotswap_1u, symbol Switch:SW_Push
- removed SW3: KEY_3 MX HOTSWAP, Workbench:keyswitch_cherrymx_hotswap_1u, symbol Switch:SW_Push
- removed SW4: KEY_4 MX HOTSWAP, Workbench:keyswitch_cherrymx_hotswap_1u, symbol Switch:SW_Push
- removed SW5: KEY_5 MX HOTSWAP, Workbench:keyswitch_cherrymx_hotswap_1u, symbol Switch:SW_Push
- removed SW6: KEY_6 MX HOTSWAP, Workbench:keyswitch_cherrymx_hotswap_1u, symbol Switch:SW_Push
- removed SW7: KEY_7 MX HOTSWAP, Workbench:keyswitch_cherrymx_hotswap_1u, symbol Switch:SW_Push
- removed SW8: KEY_8 MX HOTSWAP, Workbench:keyswitch_cherrymx_hotswap_1u, symbol Switch:SW_Push
- removed SW9: KEY_9 MX HOTSWAP, Workbench:keyswitch_cherrymx_hotswap_1u, symbol Switch:SW_Push
- removed U1: MCP23017-E/SO / 0x20, Package_SO:SOIC-28W_7.5x17.9mm_P1.27mm, symbol Interface_Expansion:MCP23017x-x-SO
Connections:
- no-connect marks 18 -> 12
Other:
- added sheet Upper (workbench-s3-r01-upper.kicad_sch)
- note added: "1 GND"
- note added: "1 x 24 / 2.54 mm"
- note added: "10k"
- note added: "2 3V3"
- note added: "3 SDA / GPIO13"
- note added: "3.3 V IO | native core-board USB-C | 4-wire cable to upper board"
- note added: "4 SCL / GPIO14"
- note added: "BOOT"
- note added: "EXPANSION / 22 SPARE GPIO"
- note added: "EXTERNAL BOOT / RESET"
- note added: "J8 pins 1-4 -> J9 pins 1-4 (1:1)"
- note added: "JST XH / 4 pins"
- note added: "Keyboard + display"
- note added: "LOWER BOARD / SOCKETED ESP32-S3"
- note added: "Normally-open buttons to GND; EN bias is on the core board."
- note added: "P1 / right socket"
- note added: "P2 / left socket"
- note added: "Pin 1 is at the antenna end. USB/PSRAM/strap pins marked NC stay unused."
- note added: "RESET"
- note added: "UPPER-BOARD CABLE"
- note added: "YD CORE BOARD / 2 x 22 SOCKETS"
- note removed: "I2C4 TWO-BOARD DRAFT: J8/J9 pins 1-4 = GND 3V3 SDA SCL. MCP23017 at 0x20 shares the OLED bus."
- note removed: "J2 matches supplied module diagram: pins 1-9 = VCC GND BAK TRB TRA PSH SCL SDA CON. VCC = 3.3V ONLY."
- note removed: "R1/R2: 2.2k I2C pull-ups; check module parallel pull-ups. GPA5-7 rows: selected LOW, inactive HIGH; diode K to row."
- note removed: "UP_* nets are on the upper board. Lower and upper nets join ONLY through the external cable; see interconnect.csv."
- title: Kivo Workbench -> Workbench S3 r01 / LOWER
- moved on the sheet: J1, J4, J5, J6, J7, J8, R3
