File: hardware/keypad-i2c-k18-r01/keypad-i2c-k18-r01.kicad_sch (KiCad schematic)
At the start: 43 parts, among them J1 I2C / 3V3 / 1x4 FEMALE / 2.54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, SW1 KEY_1 MX HOTSWAP, SW10 KEY_10 MX HOTSWAP, SW11 KEY_11 MX HOTSWAP, SW12 KEY_12 MX HOTSWAP, SW13 KEY_13 MX HOTSWAP, SW14 KEY_14 MX HOTSWAP, SW15 KEY_15 MX HOTSWAP, SW16 KEY_16 MX HOTSWAP, SW17 KEY_17 MX HOTSWAP, SW18 KEY_18 MX HOTSWAP, SW2 KEY_2 MX HOTSWAP, SW3 KEY_3 MX HOTSWAP, SW4 KEY_4 MX HOTSWAP, SW5 KEY_5 MX HOTSWAP, SW6 KEY_6 MX HOTSWAP, SW7 KEY_7 MX HOTSWAP, SW8 KEY_8 MX HOTSWAP, SW9 KEY_9 MX HOTSWAP, U1 MCP23017-E/SO / 0x20

Commit message: Update application implementation
Parts:
- C1: value 10u 10V X7R -> 10u 10V X5R; footprint Capacitor_SMD:C_0805_2012Metric_Pad1.18x1.45mm_HandSolder -> Capacitor_SMD:C_0402_1005Metric_Pad0.74x0.62mm_HandSolder
- C2: footprint Capacitor_SMD:C_0805_2012Metric_Pad1.18x1.45mm_HandSolder -> Capacitor_SMD:C_0402_1005Metric_Pad0.74x0.62mm_HandSolder
- R1, R2, R3: footprint Resistor_SMD:R_0805_2012Metric_Pad1.20x1.40mm_HandSolder -> Resistor_SMD:R_0402_1005Metric_Pad0.72x0.64mm_HandSolder
Changed lines of the file:
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@@
       )
     )
-    (property "Value" "10u 10V X7R"
+    (property "Value" "10u 10V X5R"
       (at 33.02 95.25 0)
       (hide yes)
@@
       )
     )
-    (property "Footprint" "Capacitor_SMD:C_0805_2012Metric_Pad1.18x1.45mm_HandSolder"
+    (property "Footprint" "Capacitor_SMD:C_0402_1005Metric_Pad0.74x0.62mm_HandSolder"
       (at 33.02 95.25 0)
       (hide yes)
@@
       )
     )
-    (property "Footprint" "Resistor_SMD:R_0805_2012Metric_Pad1.20x1.40mm_HandSolder"
+    (property "Footprint" "Resistor_SMD:R_0402_1005Metric_Pad0.72x0.64mm_HandSolder"
       (at 127 45.72 0)
       (hide yes)
@@
       )
     )
-    (property "Footprint" "Resistor_SMD:R_0805_2012Metric_Pad1.20x1.40mm_HandSolder"
+    (property "Footprint" "Resistor_SMD:R_0402_1005Metric_Pad0.72x0.64mm_HandSolder"
       (at 101.6 45.72 0)
       (hide yes)
@@
       )
     )
-    (property "Footprint" "Capacitor_SMD:C_0805_2012Metric_Pad1.18x1.45mm_HandSolder"
+    (property "Footprint" "Capacitor_SMD:C_0402_1005Metric_Pad0.74x0.62mm_HandSolder"
       (at 205.74 50.8 0)
       (hide yes)
@@
       )
     )
-    (property "Footprint" "Resistor_SMD:R_0805_2012Metric_Pad1.20x1.40mm_HandSolder"
+    (property "Footprint" "Resistor_SMD:R_0402_1005Metric_Pad0.72x0.64mm_HandSolder"
       (at 127 74.93 0)
       (hide yes)
